File: bms_monitor.kicad_pcb (KiCad board)
At the start: 2 copper layers, 115 x 65 mm, 238 parts, among them CN1 10nF, CN10 10nF, CN11 10nF, CN12 10nF, CN13 10nF, CN14 10nF, CN2 10nF, CN3 10nF, CN4 10nF, CN5 10nF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

Commit message: Removed logo
Parts:
- added kibuzzard-636A30EE: G***, kibuzzard-636A30EE, F.Cu at (126.5, 95.9)
- added kibuzzard-636A3124: G***, kibuzzard-636A3124, F.Cu at (126.5, 110.7)
- added kibuzzard-636A3184: G***, kibuzzard-636A3184, F.Cu at (148.6, 70.5)
- added kibuzzard-636A31C6: G***, kibuzzard-636A31C6, F.Cu at (148.6, 80.9)
