File: bms_monitor.kicad_sch (KiCad schematic)
At the start: 22 parts, among them J1 Conn_01x02, J13 Conn_ARM_JTAG_SWD_10, J2 Conn_01x02, J3 Conn_01x02, J4 Conn_01x02, U1 STM32L432KBUx, U2 MCP1812AT-033-TT, U3 DSC61XX, U4 TFBS4652

Commit message: Removed logo
Other:
- company: E-Agle TRT -> Filippo Volpe
Changed lines of the file:
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@@
   (title_block
     (title "BMS Monitor")
-    (date "2022-10-25")
-    (company "E-Agle TRT")
-    (comment 1 "Filippo Volpe")
+    (date "2022-11-08")
+    (company "Filippo Volpe")
   )
   (junction (at 152.4 190.5) (diameter 0) (color 0 0 0 0)
