File: stack.kicad_sch (KiCad schematic)
At the start: 108 parts, among them CN1 10nF, CN2 10nF, CN3 10nF, CN4 10nF, CN5 10nF, CN6 10nF, CN7 10nF, J5 CELLS, J6 TEMP0, J7 TEMP1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

Commit message: Removed logo
Other:
- company: E-Agle TRT -> Filippo Volpe
Changed lines of the file:
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@@
   (title_block
     (title "BMS Monitor")
-    (company "E-Agle TRT")
-    (comment 1 "Filippo Volpe")
+    (company "Filippo Volpe")
   )
   (junction (at 256.54 50.8) (diameter 0) (color 0 0 0 0)
